File: data-logger/data-logger.kicad_pcb (KiCad board)
At the start: 2 copper layers, 15 parts, among them J4 SM04B-GHS-TB, J5 SM04B-GHS-TB, J6 SM04B-GHS-TB, J7 Micro_SD_Card, J8 SM04B-GHS-TB, U3 MAX31855KASA, U4 MAX31855KASA, U5 MAX31855KASA

Commit message: layout
Parts:
- added C11: 0.1uF, Capacitor_SMD:C_0603_1608Metric, F.Cu at (111.8, 130.0)
- added C12: 10uF, Capacitor_SMD:C_0603_1608Metric, F.Cu at (108.2, 130.0)
- added J1: MPT-0,5-2-2.54, TerminalBlock_Phoenix:TerminalBlock_Phoenix_MPT-0,5-2-2.54_1x02_P2.54mm_Horizontal, F.Cu at (104.5, 107.2)
- added J2: MPT-0,5-2-2.54, TerminalBlock_Phoenix:TerminalBlock_Phoenix_MPT-0,5-2-2.54_1x02_P2.54mm_Horizontal, F.Cu at (104.5, 113.8)
- added J3: MPT-0,5-2-2.54, TerminalBlock_Phoenix:TerminalBlock_Phoenix_MPT-0,5-2-2.54_1x02_P2.54mm_Horizontal, F.Cu at (104.5, 120.4)
- added J9: Conn_01x04, Connector_PinSocket_2.54mm:PinSocket_1x04_P2.54mm_Vertical, F.Cu at (118.1, 79.2)
- added R1: 2K, Resistor_SMD:R_0603_1608Metric_Pad0.98x0.95mm_HandSolder, F.Cu at (114.3, 84.3)
- added R2: 2K, Resistor_SMD:R_0603_1608Metric_Pad0.98x0.95mm_HandSolder, F.Cu at (114.3, 86.8)
- added R3: 2K, Resistor_SMD:R_0603_1608Metric_Pad0.98x0.95mm_HandSolder, F.Cu at (124.5, 93.5)
- added R4: 2K, Resistor_SMD:R_0603_1608Metric_Pad0.98x0.95mm_HandSolder, F.Cu at (124.5, 96.0)
- added TP1: 5016, jannett_footprints:TestPoint_Keystone_5016_Vias, F.Cu at (155.2, 75.7)
- added TP2: 5016, jannett_footprints:TestPoint_Keystone_5016_Vias, F.Cu at (155.2, 81.3)
- added TP3: 5016, jannett_footprints:TestPoint_Keystone_5016_Vias, F.Cu at (155.2, 86.9)
- added TP4: 5016, jannett_footprints:TestPoint_Keystone_5016_Vias, F.Cu at (155.2, 92.6)
- added TP5: 5016, jannett_footprints:TestPoint_Keystone_5016_Vias, F.Cu at (155.2, 98.2)
- J7: value Micro_SD_Card -> DM3D-SF; footprint Connector_Card:microSD_HC_Molex_47219-2001 -> Connector_Card:microSD_HC_Hirose_DM3D-SF
- moved C10 70.7 mm to (101.1, 130.0)
- moved C8 70.5 mm to (104.6, 130.0)
- moved C5 67.3 mm to (115.3, 130.0)
- moved C9 60.1 mm to (110.0, 121.7), turned to 90 degrees
- moved C7 59.3 mm to (110.0, 115.1), turned to 90 degrees
- moved C6 57.5 mm to (110.0, 108.5), turned to 90 degrees
- moved J4 56.4 mm to (117.6, 94.7), turned to -90 degrees
- moved J8 50.3 mm to (110.0, 94.7), turned to -90 degrees
- moved U3 47.2 mm to (115.8, 108.7)
- moved U4 47.2 mm to (115.8, 115.3)
- moved U5 47.2 mm to (115.8, 121.9)
- moved J5 41.0 mm to (116.8, 70.6), turned to -90 degrees
- moved J6 37.0 mm to (156.0, 106.2), turned to 90 degrees
- moved J7 32.5 mm to (139.4, 133.3)
Connections:
- A1 pad 39: unconnected-(A1-VSYS-Pad39) -> Net-(A1-VSYS)
- A1 pad 4: unconnected-(A1-GPIO2-Pad4) -> SDA1
- A1 pad 40: unconnected-(A1-VBUS-Pad40) -> +5V
- A1 pad 5: unconnected-(A1-GPIO3-Pad5) -> SCL1
- A1 pad 6: SDA -> SDA0
- A1 pad 7: SCL -> SCL0
- J4 pad 1: +3.3V -> +5V
- J4 pad 2: unconnected-(J4-Pin_2-Pad2) -> SCL0
- J4 pad 3: unconnected-(J4-Pin_3-Pad3) -> SDA0
- J5 pad 1: +3.3V -> +5V
- J5 pad 2: unconnected-(J5-Pin_2-Pad2) -> TX
- J5 pad 3: unconnected-(J5-Pin_3-Pad3) -> RX
- J7 pad 9: unconnected-(J7-SHIELD-Pad9) -> GND
- J8 pad 1: +3.3V -> +5V
- J8 pad 2: unconnected-(J8-Pin_2-Pad2) -> SCL0
- J8 pad 3: unconnected-(J8-Pin_3-Pad3) -> SDA0

Commit message: layout
Parts:
- added H1: MountingHole, MountingHole:MountingHole_3.2mm_M3, F.Cu at (105.2, 74.7)
- added H2: MountingHole, MountingHole:MountingHole_3.2mm_M3, F.Cu at (156.5, 74.7)
- added H3: MountingHole, MountingHole:MountingHole_3.2mm_M3, F.Cu at (156.5, 136.1)
- added H4: MountingHole, MountingHole:MountingHole_3.2mm_M3, F.Cu at (105.2, 136.1)
- added R5: 0, Resistor_SMD:R_0603_1608Metric_Pad0.98x0.95mm_HandSolder, F.Cu at (114.8, 84.4)
- added R6: 0, Resistor_SMD:R_0603_1608Metric_Pad0.98x0.95mm_HandSolder, F.Cu at (124.2, 84.3)
- moved TP3 61.1 mm to (114.6, 132.6)
- moved TP5 48.4 mm to (121.2, 132.6)
- moved C10 23.8 mm to (116.6, 112.0)
- moved C12 20.4 mm to (127.8, 135.9), turned to -90 degrees
- moved C11 19.7 mm to (130.6, 135.9), turned to -90 degrees
- moved J5 19.2 mm to (104.9, 85.6)
- moved C8 15.8 mm to (116.6, 119.6)
- moved TP2 15.8 mm to (156.7, 97.0)
- moved TP1 14.1 mm to (156.7, 89.7)
- moved TP4 10.4 mm to (156.7, 82.3)
- moved R2 10.2 mm to (124.2, 89.4), turned to 180 degrees
- moved R1 10.2 mm to (124.2, 86.9), turned to 180 degrees
- moved J8 5.80 mm to (104.9, 97.5)
- moved C5 3.07 mm to (116.6, 127.3)
- moved C9 2.90 mm to (112.3, 123.4)
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Connections:
- J9 pad 2: +3.3V -> Net-(J9-Pin_2)
Other:
- board outline added: 58.4 x 68.6 mm
- board text added: "1 5V 2 ADC1 3 ADC0 4 GND"
- board text added: "1 5V 2 SCL 3 SDA 4 GND"
- board text added: "1 5V 2 TX 3 RX 4 GND"
- board text added: "3.3V"
- board text added: "5V"
- board text added: "GND"
- board text added: "Install for 3.3V"
- board text added: "Install for 5V"
- board text added: "R- Y+"
- board text added: "VSYS"
