File: data-logger/data-logger.kicad_pcb (KiCad board)
At the start: 2 copper layers, 58.4 x 68.6 mm, 36 parts, among them J1 MPT-0,5-2-2.54, J2 MPT-0,5-2-2.54, J3 MPT-0,5-2-2.54, J4 SM04B-GHS-TB, J5 SM04B-GHS-TB, J6 SM04B-GHS-TB, J7 DM3D-SF, J8 SM04B-GHS-TB, J9 Conn_01x04, U3 MAX31855KASA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

Commit message: finished
Routing:
- net +3.3V: track 0.00 -> 171.5 mm
- net +5V: track 0.00 -> 96.6 mm
- net MISO1: track 0.00 -> 31.6 mm
- net SDA0: track 0.00 -> 31.2 mm, vias 0 -> 1
- net CS3: track 0.00 -> 31.0 mm, vias 0 -> 1
- net MOSI0: track 0.00 -> 29.3 mm
- net CS0: track 0.00 -> 29.0 mm
- net SCK1: track 0.00 -> 28.6 mm
- net TX: track 0.00 -> 28.2 mm
- net SCL0: track 0.00 -> 28.1 mm, vias 0 -> 1
- net SCK0: track 0.00 -> 27.9 mm, vias 0 -> 1
- net RX: track 0.00 -> 27.7 mm
- net GND: track 0.00 -> 24.3 mm, vias 0 -> 13
- net MISO0: track 0.00 -> 23.4 mm, vias 0 -> 1
- net SDA1: track 0.00 -> 22.1 mm
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- added copper zone on B.Cu, net GND
Other:
- board text added: "Data Logger V01"
- board text added: "Jannett W"
