File: data-logger/data-logger.kicad_sch (KiCad schematic)
At the start: 3 parts, among them J7 Micro_SD_Card, U1 ATmega328PB-A, U2 MAX31855KASA

Commit message: sch
Parts:
- removed U1: ATmega328PB-A, Package_QFP:TQFP-32_7x7mm_P0.8mm, symbol MCU_Microchip_ATmega:ATmega328PB-A
- removed U2: MAX31855KASA, Package_SO:SOIC-8_3.9x4.9mm_P1.27mm, symbol Sensor_Temperature:MAX31855KASA
- added A1: RaspberryPi_Pico, Module:RaspberryPi_Pico_Common_Unspecified, symbol MCU_Module:RaspberryPi_Pico
- added C10, C5, C8: 0.1uF, Capacitor_SMD:C_0603_1608Metric, symbol Device:C_Small
- added C6, C7, C9: 10nF, Capacitor_SMD:C_0603_1608Metric, symbol Device:C_Small
- added J4, J5, J6, J8: SM04B-GHS-TB, Connector_JST:JST_GH_SM04B-GHS-TB_1x04-1MP_P1.25mm_Horizontal, symbol Connector_Generic:Conn_01x04
- added TC1, TC2, TC3: Thermocouple_Block, symbol Device:Thermocouple_Block
- added U3, U4, U5: MAX31855KASA, Package_SO:SOIC-8_3.9x4.9mm_P1.27mm, symbol Sensor_Temperature:MAX31855KASA
Connections:
- net CS0: now reaches J7.2 (DAT3/CD)
- net CS0: now also A1.22 (GPIO17)
- net MOSI0: now reaches J7.3 (CMD)
- net MOSI0: now also A1.25 (GPIO19)
- net +3.3V: now reaches J7.4 (VDD)
- net +3.3V: now also A1.36 (3V3), C10.1, C5.1, C8.1, J4.1 (Pin_1), J5.1 (Pin_1), J6.1 (Pin_1), J8.1 (Pin_1), U3.4 (V_{CC}), U4.4 (V_{CC}), U5.4 (V_{CC})
- net SCK0: now reaches J7.5 (CLK)
- net SCK0: now also A1.24 (GPIO18)
- net GND: now reaches J7.6 (VSS)
- net GND: now also A1.13 (GND), A1.18 (GND), A1.23 (GND), A1.28 (GND), A1.3 (GND), A1.33 (AGND), A1.38 (GND), A1.8 (GND), C10.2, C5.2, C8.2, J4.4 (Pin_4), J5.4 (Pin_4), J6.4 (Pin_4), J8.4 (Pin_4), U3.1 (GND), U4.1 (GND), U5.1 (GND)
- net MISO0: now reaches J7.7 (DAT0)
- net MISO0: now also A1.21 (GPIO16)
- new net: C9.2, TC3.2 (-), U5.2 (T-)
- new net: C9.1, TC3.1 (+), U5.3 (T+)
- new net: C6.1, TC1.1 (+), U3.3 (T+)
- new net: C6.2, TC1.2 (-), U3.2 (T-)
- new net: C7.1, TC2.1 (+), U4.3 (T+)
- new net: C7.2, TC2.2 (-), U4.2 (T-)
- new net ADC0: A1.31 (GPIO26_ADC0), J6.2 (Pin_2)
- new net ADC1: A1.32 (GPIO27_ADC1), J6.3 (Pin_3)
- new net CS1: A1.17 (GPIO13), U3.6 (~{CS})
- new net CS2: A1.12 (GPIO9), U4.6 (~{CS})
- new net CS3: A1.11 (GPIO8), U5.6 (~{CS})
- new net MISO1: A1.16 (GPIO12), U3.7 (SO), U4.7 (SO), U5.7 (SO)
- new net RX: A1.2 (GPIO1)
- new net SCK1: A1.19 (GPIO14), U3.5 (SCK), U4.5 (SCK), U5.5 (SCK)
- new net SCL: A1.7 (GPIO5)
- new net SDA: A1.6 (GPIO4)
- new net TX: A1.1 (GPIO0)
Other:
- note added: "Analog"
- note added: "I2C"
- note added: "UART"
- moved on the sheet: J7

Commit message: layout
Parts:
- added C11: 0.1uF, Capacitor_SMD:C_0603_1608Metric, symbol Device:C_Small
- added C12: 10uF, Capacitor_SMD:C_0603_1608Metric, symbol Device:C_Small
- added J1, J2, J3: MPT-0,5-2-2.54, TerminalBlock_Phoenix:TerminalBlock_Phoenix_MPT-0,5-2-2.54_1x02_P2.54mm_Horizontal, symbol Connector:Screw_Terminal_01x02
- added J9: Conn_01x04, Connector_PinSocket_2.54mm:PinSocket_1x04_P2.54mm_Vertical, symbol Connector_Generic:Conn_01x04
- added R1, R2, R3, R4: 2K, Resistor_SMD:R_0603_1608Metric_Pad0.98x0.95mm_HandSolder, symbol Device:R_US
- added TP1, TP2, TP3, TP4, TP5: 5016, jannett_footprints:TestPoint_Keystone_5016_Vias, symbol Connector:TestPoint
- J7: value Micro_SD_Card -> DM3D-SF; footprint Connector_Card:microSD_HC_Molex_47219-2001 -> Connector_Card:microSD_HC_Hirose_DM3D-SF
Connections:
- net SCL is gone; now on net SCL0: A1.7 (GPIO5)
- net SDA is gone; now on net SDA0: A1.6 (GPIO4)
- net +3.3V: now also C11.1, C12.1, J9.2 (Pin_2), R1.1, R2.1, R3.1, R4.1, TP5.1; no longer J4.1 (Pin_1), J5.1 (Pin_1), J8.1 (Pin_1)
- net GND: now also J7.9 (SHIELD), C11.2, C12.2, J9.1 (Pin_1), TP2.1, TP3.1
- net RX: now also J5.3 (Pin_3)
- net TX: now also J5.2 (Pin_2)
- net at A1.39 (VSYS): now also TP1.1
- net SDA1: now reaches A1.4 (GPIO2)
- net SDA1: now also J9.4 (Pin_4), R2.2
- net +5V: now reaches A1.40 (VBUS)
- net +5V: now also J4.1 (Pin_1), J5.1 (Pin_1), J8.1 (Pin_1), TP4.1
- net SCL1: now reaches A1.5 (GPIO3)
- net SCL1: now also J9.3 (Pin_3), R1.2
- net at C9.2, TC3.2 (-), U5.2 (T-): now also J3.1 (Pin_1)
- net at C9.1, TC3.1 (+), U5.3 (T+): now also J3.2 (Pin_2)
- net at C6.1, TC1.1 (+), U3.3 (T+): now also J1.2 (Pin_2)
- net at C6.2, TC1.2 (-), U3.2 (T-): now also J1.1 (Pin_1)
- net SCL0: now reaches J8.2 (Pin_2)
- net SCL0: now also J4.2 (Pin_2), R3.2
- net SDA0: now reaches J8.3 (Pin_3)
- net SDA0: now also J4.3 (Pin_3), R4.2
- net at C7.1, TC2.1 (+), U4.3 (T+): now also J2.2 (Pin_2)
- net at C7.2, TC2.2 (-), U4.2 (T-): now also J2.1 (Pin_1)

Commit message: layout
Parts:
- added H1, H2, H3, H4: MountingHole, MountingHole:MountingHole_3.2mm_M3, symbol Mechanical:MountingHole
- added R5, R6: 0, Resistor_SMD:R_0603_1608Metric_Pad0.98x0.95mm_HandSolder, symbol Device:R_US
Connections:
- net +3.3V: now also R6.1; no longer J9.2 (Pin_2)
- net +5V: now also R5.1
- new net: J9.2 (Pin_2), R5.2, R6.2
Other:
- moved on the sheet: J9
